File: Arduino_CQbrushless.kicad_sch (KiCad schematic)
At the start: 14 parts, among them J1 Nucleo_F302R8, J2 AE-LLCNV8-DIP20, J3 AE-LLCNV8-DIP20, J4 Conn_01x03, J6 Conn_01x04

Commit message: 0122
Connections:
- net GND: now also J1.19 (Pin_19), J1.20 (Pin_20), J1.22 (Pin_22), J1.47, J1.58, J1.70, J1.8 (Pin_8)
Changed lines of the file:
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@@
   (junction (at 126.365 113.665) (diameter 0) (color 0 0 0 0)
   )
+  (junction (at 196.85 67.945) (diameter 0) (color 0 0 0 0)
+  )
   (junction (at 138.43 165.1) (diameter 0) (color 0 0 0 0)
   )
@@
   (junction (at 121.285 106.045) (diameter 0) (color 0 0 0 0)
   )
+  (junction (at 115.57 52.705) (diameter 0) (color 0 0 0 0)
+  )
   (junction (at 48.26 149.225) (diameter 0) (color 0 0 0 0)
   )
@@
   )
   (junction (at 113.665 103.505) (diameter 0) (color 0 0 0 0)
+  )
+  (junction (at 159.385 40.005) (diameter 0) (color 0 0 0 0)
   )
   (junction (at 113.665 93.345) (diameter 0) (color 0 0 0 0)
@@
     (stroke (width 0) (type default))
   )
+  (wire (pts (xy 196.85 67.945) (xy 196.85 68.58))
+    (stroke (width 0) (type default))
+  )
   (wire (pts (xy 19.685 144.145) (xy 44.45 144.145))
     (stroke (width 0) (type default))
@@
     (stroke (width 0) (type default))
   )
+  (wire (pts (xy 97.155 52.705) (xy 102.87 52.705))
+    (stroke (width 0) (type default))
+  )
   (wire (pts (xy 115.57 50.165) (xy 123.825 50.165))
     (stroke (width 0) (type default))
@@
     (stroke (width 0) (type default))
   )
+  (wire (pts (xy 163.83 40.005) (xy 159.385 40.005))
+    (stroke (width 0) (type default))
+  )
   (wire (pts (xy 39.37 91.44) (xy 45.085 91.44))
     (stroke (width 0) (type default))
@@
     (stroke (width 0) (type default))
   )
+  (wire (pts (xy 115.57 52.705) (xy 120.65 52.705))
+    (stroke (width 0) (type default))
+  )
   (wire (pts (xy 126.365 113.665) (xy 126.365 117.475))
     (stroke (width 0) (type default))
@@
     (stroke (width 0) (type default))
   )
+  (wire (pts (xy 176.53 52.705) (xy 196.85 52.705))
+    (stroke (width 0) (type default))
+  )
   (wire (pts (xy 115.57 75.565) (xy 123.19 75.565))
     (stroke (width 0) (type default))
@@
     (stroke (width 0) (type default))
   )
+  (wire (pts (xy 159.385 40.005) (xy 159.385 42.545))
+    (stroke (width 0) (type default))
+  )
   (wire (pts (xy 35.56 155.575) (xy 39.37 155.575))
     (stroke (width 0) (type default))
@@
     (stroke (width 0) (type default))
   )
+  (wire (pts (xy 176.53 67.945) (xy 196.85 67.945))
+    (stroke (width 0) (type default))
+  )
   (wire (pts (xy 35.56 155.575) (xy 35.56 121.285))
     (stroke (width 0) (type default))
@@
     (stroke (width 0) (type default))
   )
+  (wire (pts (xy 115.57 37.465) (xy 159.385 37.465))
+    (stroke (width 0) (type default))
+  )
   (wire (pts (xy 132.715 128.27) (xy 145.415 128.27))
     (stroke (width 0) (type default))
@@
     (stroke (width 0) (type default))
   )
+  (wire (pts (xy 159.385 37.465) (xy 159.385 40.005))
+    (stroke (width 0) (type default))
+  )
   (wire (pts (xy 20.955 23.495) (xy 20.955 141.605))
     (stroke (width 0) (type default))
@@
     (stroke (width 0) (type default))
   )
+  (wire (pts (xy 115.57 52.705) (xy 115.57 55.245))
+    (stroke (width 0) (type default))
+  )
   (wire (pts (xy 123.825 125.095) (xy 123.825 128.27))
     (stroke (width 0) (type default))
   )
   (wire (pts (xy 48.26 149.225) (xy 48.26 151.765))
+    (stroke (width 0) (type default))
+  )
+  (wire (pts (xy 196.85 52.705) (xy 196.85 67.945))
     (stroke (width 0) (type default))
   )
@@
         (path "/e7502d87-1b50-48ec-aa02-3ff7ae62932a"
           (reference "#PWR05") (unit 1)
+        )
+      )
+    )
+  )
+  (symbol (lib_id "power:GND") (at 196.85 68.58 0) (unit 1)
+    (in_bom yes) (on_board yes) (dnp no) (fields_autoplaced)
+    (property "Reference" "#PWR010" (at 196.85 74.93 0)
+      (effects (font (size 1.27 1.27)) hide)
+    )
+    (property "Value" "GND" (at 196.85 73.66 0)
+      (effects (font (size 1.27 1.27)))
+    )
+    (property "Footprint" "" (at 196.85 68.58 0)
+      (effects (font (size 1.27 1.27)) hide)
+    )
+    (property "Datasheet" "" (at 196.85 68.58 0)
+      (effects (font (size 1.27 1.27)) hide)
+    )
+    (pin "1")
+    (instances
+      (project "Arduino_CQbrushless"
+        (path "/e7502d87-1b50-48ec-aa02-3ff7ae62932a"
+          (reference "#PWR010") (unit 1)
         )
       )
@@
     )
   )
+  (symbol (lib_id "power:GND") (at 159.385 42.545 0) (unit 1)
+    (in_bom yes) (on_board yes) (dnp no) (fields_autoplaced)
+    (property "Reference" "#PWR012" (at 159.385 48.895 0)
+      (effects (font (size 1.27 1.27)) hide)
+    )
+    (property "Value" "GND" (at 159.385 46.99 0)
+      (effects (font (size 1.27 1.27)))
+    )
+    (property "Footprint" "" (at 159.385 42.545 0)
+      (effects (font (size 1.27 1.27)) hide)
+    )
+    (property "Datasheet" "" (at 159.385 42.545 0)
+      (effects (font (size 1.27 1.27)) hide)
+    )
+    (pin "1")
+    (instances
+      (project "Arduino_CQbrushless"
+        (path "/e7502d87-1b50-48ec-aa02-3ff7ae62932a"
+          (reference "#PWR012") (unit 1)
+        )
+      )
+    )
+  )
   (symbol (lib_id "power:+3.3V") (at 144.78 138.43 0) (unit 1)
     (in_bom yes) (on_board yes) (dnp no)
@@
         (path "/e7502d87-1b50-48ec-aa02-3ff7ae62932a"
           (reference "#PWR02") (unit 1)
+        )
+      )
+    )
+  )
+  (symbol (lib_id "power:GND") (at 120.65 52.705 0) (unit 1)
+    (in_bom yes) (on_board yes) (dnp no)
+    (property "Reference" "#PWR013" (at 120.65 59.055 0)
+      (effects (font (size 1.27 1.27)) hide)
+    )
+    (property "Value" "GND" (at 121.92 55.88 0)
+      (effects (font (size 1.27 1.27)))
+    )
+    (property "Footprint" "" (at 120.65 52.705 0)
+      (effects (font (size 1.27 1.27)) hide)
+    )
+    (property "Datasheet" "" (at 120.65 52.705 0)
+      (effects (font (size 1.27 1.27)) hide)
+    )
+    (pin "1")
+    (instances
+      (project "Arduino_CQbrushless"
+        (path "/e7502d87-1b50-48ec-aa02-3ff7ae62932a"
+          (reference "#PWR013") (unit 1)
         )
       )
@@
         )
       )
+    )
+  )
+  (symbol (lib_id "power:GND") (at 97.155 52.705 0) (unit 1)
+    (in_bom yes) (on_board yes) (dnp no) (fields_autoplaced)
+    (property "Reference" "#PWR014" (at 97.155 59.055 0)
+      (effects (font (size 1.27 1.27)) hide)
+    )
+    (property "Value" "GND" (at 97.155 57.15 0)
+      (effects (font (size 1.27 1.27)))
+    )
+    (property "Footprint" "" (at 97.155 52.705 0)
+      (effects (font (size 1.27 1.27)) hide)
+    )
+    (property "Datasheet" "" (at 97.155 52.705 0)
+      (effects (font (size 1.27 1.27)) hide)
+    )
+    (pin "1")
+    (instances
+      (project "Arduino_CQbrushless"
+        (path "/e7502d87-1b50-48ec-aa02-3ff7ae62932a"
+          (reference "#PWR014") (unit 1)
+        )
+      )

Commit message: ver0.3
Parts:
- removed R7, R8: R, Resistor_THT:R_Axial_DIN0309_L9.0mm_D3.2mm_P12.70mm_Horizontal, symbol Device:R
Connections:
- net at A1.A3: now also J1.30 (Pin_30)
Changed lines of the file:
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@@
   (junction (at 138.43 165.1) (diameter 0) (color 0 0 0 0)
   )
-  (junction (at 39.37 155.575) (diameter 0) (color 0 0 0 0)
-  )
   (junction (at 121.285 106.045) (diameter 0) (color 0 0 0 0)
   )
@@
   (junction (at 116.205 93.345) (diameter 0) (color 0 0 0 0)
   )
-  (junction (at 45.72 163.83) (diameter 0) (color 0 0 0 0)
-  )
   (junction (at 113.665 103.505) (diameter 0) (color 0 0 0 0)
   )
@@
   )
   (junction (at 113.665 93.345) (diameter 0) (color 0 0 0 0)
-  )
-  (junction (at 39.37 139.065) (diameter 0) (color 0 0 0 0)
   )
   (junction (at 132.715 93.345) (diameter 0) (color 0 0 0 0)
@@
     (stroke (width 0) (type default))
   )
+  (wire (pts (xy 115.57 65.405) (xy 127 65.405))
+    (stroke (width 0) (type default))
+  )
   (wire (pts (xy 115.57 50.165) (xy 123.825 50.165))
     (stroke (width 0) (type default))
@@
     (stroke (width 0) (type default))
   )
-  (wire (pts (xy 39.37 156.21) (xy 39.37 155.575))
-    (stroke (width 0) (type default))
-  )
   (wire (pts (xy 99.06 111.125) (xy 106.68 111.125))
     (stroke (width 0) (type default))
@@
     (stroke (width 0) (type default))
   )
+  (wire (pts (xy 15.875 19.05) (xy 15.875 121.285))
+    (stroke (width 0) (type default))
+  )
   (wire (pts (xy 132.715 128.27) (xy 126.365 128.27))
     (stroke (width 0) (type default))
@@
     (stroke (width 0) (type default))
   )
-  (wire (pts (xy 35.56 155.575) (xy 39.37 155.575))
-    (stroke (width 0) (type default))
-  )
   (wire (pts (xy 154.305 70.485) (xy 163.83 70.485))
     (stroke (width 0) (type default))
@@
     (stroke (width 0) (type default))
   )
-  (wire (pts (xy 39.37 163.83) (xy 45.72 163.83))
-    (stroke (width 0) (type default))
-  )
   (wire (pts (xy 145.415 106.045) (xy 151.13 106.045))
     (stroke (width 0) (type default))
@@
     (stroke (width 0) (type default))
   )
-  (wire (pts (xy 35.56 155.575) (xy 35.56 121.285))
+  (wire (pts (xy 127 19.05) (xy 15.875 19.05))
     (stroke (width 0) (type default))
   )
@@
     (stroke (width 0) (type default))
   )
+  (wire (pts (xy 127 65.405) (xy 127 19.05))
+    (stroke (width 0) (type default))
+  )
   (wire (pts (xy 159.385 37.465) (xy 159.385 40.005))
     (stroke (width 0) (type default))
@@
     (stroke (width 0) (type default))
   )
-  (wire (pts (xy 45.72 149.225) (xy 45.72 163.83))
+  (wire (pts (xy 45.72 149.225) (xy 45.72 164.465))
     (stroke (width 0) (type default))
   )
@@
     (stroke (width 0) (type default))
   )
-  (wire (pts (xy 22.225 139.065) (xy 39.37 139.065))
-    (stroke (width 0) (type default))
-  )
   (wire (pts (xy 163.83 60.325) (xy 159.385 60.325))
     (stroke (width 0) (type default))
@@
     (stroke (width 0) (type default))
   )
-  (wire (pts (xy 45.72 163.83) (xy 45.72 164.465))
-    (stroke (width 0) (type default))
-  )
   (wire (pts (xy 115.57 52.705) (xy 115.57 55.245))
     (stroke (width 0) (type default))
@@
     (stroke (width 0) (type default))
   )
-  (wire (pts (xy 39.37 139.065) (xy 39.37 147.955))
-    (stroke (width 0) (type default))
-  )
   (wire (pts (xy 145.415 99.06) (xy 145.415 100.965))
     (stroke (width 0) (type default))
@@
     (stroke (width 0) (type default))
   )
-  (wire (pts (xy 35.56 121.285) (xy 48.26 121.285))
+  (wire (pts (xy 15.875 121.285) (xy 48.26 121.285))
     (stroke (width 0) (type default))
   )
@@
     (stroke (width 0) (type default))
   )
-  (wire (pts (xy 39.37 139.065) (xy 48.26 139.065))
+  (wire (pts (xy 22.225 139.065) (xy 48.26 139.065))
     (stroke (width 0) (type default))
   )
@@
         (path "/e7502d87-1b50-48ec-aa02-3ff7ae62932a"
           (reference "#PWR010") (unit 1)
-        )
-      )
-    )
-  )
-  (symbol (lib_id "Device:R") (at 39.37 160.02 0) (unit 1)
-    (in_bom yes) (on_board yes) (dnp no)
-    (property "Reference" "R8" (at 39.37 161.29 90)
-      (effects (font (size 1.27 1.27)) (justify left))
-    )
-    (property "Value" "R" (at 41.91 161.29 0)
-      (effects (font (size 1.27 1.27)) (justify left) hide)
-    )
-    (property "Footprint" "Resistor_THT:R_Axial_DIN0309_L9.0mm_D3.2mm_P12.70mm_Horizontal" (at 37.592 160.02 90)
-      (effects (font (size 1.27 1.27)) hide)
-    )
-    (property "Datasheet" "~" (at 39.37 160.02 0)
-      (effects (font (size 1.27 1.27)) hide)
-    )
-    (pin "1")
-    (pin "2")
-    (instances
-      (project "Arduino_CQbrushless"
-        (path "/e7502d87-1b50-48ec-aa02-3ff7ae62932a"
-          (reference "R8") (unit 1)
         )
       )
@@
         )
       )
-    )
-  )
-  (symbol (lib_id "Device:R") (at 39.37 151.765 0) (unit 1)
-    (in_bom yes) (on_board yes) (dnp no)
-    (property "Reference" "R7" (at 39.37 153.035 90)
-      (effects (font (size 1.27 1.27)) (justify left))
-    )
-    (property "Value" "R" (at 41.91 153.035 0)
-      (effects (font (size 1.27 1.27)) (justify left) hide)
-    )
-    (property "Footprint" "Resistor_THT:R_Axial_DIN0309_L9.0mm_D3.2mm_P12.70mm_Horizontal" (at 37.592 151.765 90)
-      (effects (font (size 1.27 1.27)) hide)
-    )
-    (property "Datasheet" "~" (at 39.37 151.765 0)
-      (effects (font (size 1.27 1.27)) hide)
-    )
-    (pin "1")
-    (pin "2")
-    (instances
-      (project "Arduino_CQbrushless"
-        (path "/e7502d87-1b50-48ec-aa02-3ff7ae62932a"
-          (reference "R7") (unit 1)
-        )
-      )

Commit message: 0209
Parts:
- removed J2, J3: AE-LLCNV8-DIP20, Library:AE-LLCNV8-DIP, symbol New_Library:AE-LLCNV8-DIP20
Connections:
- net Direction is gone; now on net Dir_5V: J1.41
- net HU_5V is gone; now on net HU: A1.D2
- net HV_5V is gone; now on net HV: A1.D3
- net HW_5V is gone; now on net HW: A1.D1 (D1/TX)
- net Un_5V is gone; now on net Un: A1.D4, R1.2
- net Up_5V is gone; now on net Up: A1.D5, R4.1
- net Vn_5V is gone; now on net Vn: A1.D13, R2.2
- net Vp_5V is gone; now on net Vp: A1.D10, R6.1
- net Wn_5V is gone; now on net Wn: A1.D8, R3.2
- net Wp_5V is gone; now on net Wp: A1.D9, R5.1
- net +5V: now also A1.AREF, J1.16 (Pin_16)
- removed net +3.3V: A1.3V3 (3.3V), A1.AREF, J1.16 (Pin_16)
- no-connect marks 13 -> 1

Commit message: ver 0.4 (add LDO)
Parts:
- added IC1: AZ1084CD-5.0TRG1, AZ1084CD50TRG1, symbol samacsys:AZ1084CD-5.0TRG1
Connections:
- net +5V: now also R1.2, R2.2, R3.2, IC1.2 (OUTPUT); no longer A1.5V1 (5V), R1.1, R2.1, R3.1
- net GND: now also IC1.1 (GND)
- net Un: now also R1.1; no longer R1.2
- net VIN: now also IC1.3 (INPUT)
- net Vn: now also R2.1; no longer R2.2
- net Wn: now also R3.1; no longer R3.2
- net BATT: now reaches A1.A3, J1.30 (Pin_30)
- net Dir_5V renamed Dir
Other:
- moved on the sheet: J4, R1, R2, R3, R4, R5, R6

Commit message: 0214
Parts:
- added J2: Conn_01x06_Socket, Connector_PinHeader_2.54mm:PinHeader_1x06_P2.54mm_Vertical, symbol Connector:Conn_01x06_Socket
- added SW1, SW2: SW_SPDT, Connector_PinHeader_2.54mm:PinHeader_1x03_P2.54mm_Vertical, symbol Switch:SW_SPDT
- added TP1: TestPoint, TestPoint:TestPoint_Pad_D1.5mm, symbol Connector:TestPoint
- IC1: footprint AZ1084CD50TRG1 -> samacsys:AZ1084CD50TRG1
Connections:
- net BATT: now also TP1.1
- net GND: now also A1.GND4 (SPI_GND), J2.1 (Pin_1), SW1.1 (A), SW2.1 (A)
- net at A1.5V2 (SPI_5V): now also J2.2 (Pin_2)
- net at A1.D11: now also SW1.2 (B)
- net at A1.D12: now also SW2.2 (B)
- net at A1.MISO (SPI_MISO): now also J2.6 (Pin_6)
- net at A1.MOSI (SPI_MOSI): now also J2.5 (Pin_5)
- net at A1.RST2 (SPI_RESET): now also J2.3 (Pin_3)
- net at A1.SCK (SPI_SCK): now also J2.4 (Pin_4)
Other:
- moved on the sheet: R1, R2, R3, R4, R5, R6

Commit message: 0220
Parts:
- added C1, C3: C, Capacitor_SMD:C_0603_1608Metric_Pad1.08x0.95mm_HandSolder, symbol Device:C
- added C2, C4: C_Polarized, Capacitor_THT:CP_Radial_D8.0mm_P3.50mm, symbol Device:C_Polarized
- added J3: Conn_01x01_Pin, Connector_PinHeader_2.54mm:PinHeader_1x01_P2.54mm_Vertical, symbol Connector:Conn_01x01_Pin
- added JP1: SolderJumper_2_Bridged, Jumper:SolderJumper-2_P1.3mm_Bridged_Pad1.0x1.5mm, symbol Jumper:SolderJumper_2_Bridged
- added R7: R, Resistor_SMD:R_0603_1608Metric_Pad0.98x0.95mm_HandSolder, symbol Device:R
Connections:
- net +5V: now also C1.1, C2.1
- net ACCEL: now also J3.1 (Pin_1), JP1.2 (B); no longer A1.A0
- net GND: now also C1.2, C2.2, C3.2, C4.2, R7.1
- net VIN: now also C3.1, C4.1
- new net: A1.A0, JP1.1 (A), R7.2

Commit message: 0416
Parts:
- C1: footprint Capacitor_SMD:C_0603_1608Metric_Pad1.08x0.95mm_HandSolder -> Capacitor_SMD:C_0805_2012Metric_Pad1.18x1.45mm_HandSolder
