File: Arduino_CQbrushless.kicad_pcb (KiCad board)
At the start: 2 copper layers, 70.4 x 81.8 mm, 3 parts, among them J1 Nucleo_F302R8, J2 AE-LLCNV8-DIP20

Commit message: 1228
Parts:
- added J3: AE-LLCNV8-DIP20, Library:AE-LLCNV8-DIP, F.Cu at (129.1, 137.4)
- added J4: Conn_01x04, Connector_PinHeader_2.54mm:PinHeader_1x04_P2.54mm_Vertical, F.Cu at (147.0, 95.4)
- added J5: Conn_01x02, Connector_PinHeader_2.54mm:PinHeader_1x02_P2.54mm_Vertical, F.Cu at (147.0, 101.6)
- added J6: Conn_01x04, Connector_PinHeader_2.54mm:PinHeader_1x04_P2.54mm_Vertical, F.Cu at (148.3, 160.1)
- moved J2 36.7 mm to (133.1, 114.6), turned to -90 degrees
- moved A1 0.53 mm to (143.8, 157.7)
Connections:
- A1 pad 3V3: /+3.3V -> +3.3V
- A1 pad 5V1: /+5V -> +5V
- A1 pad AREF: /+3.3V -> +3.3V
- A1 pad D0: unconnected-(A1-D0/RX-PadD0) -> Net-(A1-D0/RX)
- A1 pad D1: unconnected-(A1-D1/TX-PadD1) -> Net-(A1-D1/TX)
- A1 pad D10: Net-(J2-A7) -> Net-(J3-A3)
- A1 pad D11: Net-(J2-GND) -> Net-(J3-A2)
- A1 pad D12: unconnected-(A1-PadD12) -> Net-(J3-A1)
- A1 pad D13: unconnected-(A1-PadD13) -> Net-(J3-A0)
- A1 pad D2: Net-(J2-VA) -> Net-(J2-A5)
- A1 pad D3: Net-(J2-A0) -> Net-(J2-A4)
- A1 pad D4: Net-(J2-A1) -> Net-(J5-Pin_1)
- A1 pad D5: Net-(J2-A2) -> Net-(J5-Pin_2)
- A1 pad D6: Net-(J2-A3) -> Net-(J2-A0)
- A1 pad D7: Net-(J2-A4) -> Net-(J2-A2)
- A1 pad D8: Net-(J2-A5) -> Net-(J2-A3)
- A1 pad D9: Net-(J2-A6) -> Net-(J2-A1)
- A1 pad SCL: unconnected-(A1-PadSCL) -> Net-(J6-Pin_2)
- A1 pad SDA: unconnected-(A1-PadSDA) -> Net-(J6-Pin_3)
- J1 pad 16: /+3.3V -> +3.3V
- J1 pad 18: /+5V -> +5V
- J2 pad 1: Net-(J2-VA) -> +5V
- J2 pad 10: Net-(J2-GND) -> GND
- J2 pad 11: /T_HIN -> GND
- J2 pad 12: /_R_LIN -> unconnected-(J2-B7-Pad12)
- J2 pad 13: /R_HIN -> unconnected-(J2-B6-Pad13)
- J2 pad 14: /_T_LIN -> /_S_LIN
- J2 pad 15: /S_HIN -> /T_HIN
- J2 pad 16: /_S_LIN -> /_T_LIN
- J2 pad 17: /Direction -> /_R_LIN
- J2 pad 18: /HV -> /R_HIN
- J2 pad 19: /HW -> /S_HIN
- J2 pad 20: /HU -> +3.3V
- J2 pad 8: Net-(J2-A6) -> unconnected-(J2-A6-Pad8)
- J2 pad 9: Net-(J2-A7) -> unconnected-(J2-A7-Pad9)
Routing:
- net +3.3V: track 0.00 -> 238.0 mm, vias 0 -> 1
- net Net-(A1-PadA3): track 0.00 -> 137.3 mm
- net Net-(A1-PadA4): track 0.00 -> 128.9 mm, vias 0 -> 1
- net +5V: track 0.00 -> 103.1 mm
- net /HU: track 0.00 -> 86.0 mm
- net /ACCEL: track 0.00 -> 69.9 mm
- net /S_sense: track 0.00 -> 61.7 mm
- net /T_sense: track 0.00 -> 58.7 mm, vias 0 -> 1
- net /R_sense: track 0.00 -> 55.6 mm
- net /Direction: track 0.00 -> 53.8 mm
- net /_T_LIN: track 0.00 -> 51.3 mm
- net /_S_LIN: track 0.00 -> 51.3 mm
- net /T_HIN: track 0.00 -> 45.1 mm
- net /_R_LIN: track 0.00 -> 39.2 mm
- net /HW: track 0.00 -> 35.6 mm
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- added copper zone on B.Cu, net GND
- added copper zone on F.Cu, net GND
Other:
- board size 70.4 x 81.8 mm -> 72.6 x 85.1 mm

Commit message: 0109
Parts:
- removed J5: Conn_01x02, Connector_PinHeader_2.54mm:PinHeader_1x02_P2.54mm_Vertical
- added R1: R, Resistor_THT:R_Axial_DIN0309_L9.0mm_D3.2mm_P12.70mm_Horizontal, F.Cu at (128.7, 91.0)
- added R2: R, Resistor_THT:R_Axial_DIN0309_L9.0mm_D3.2mm_P12.70mm_Horizontal, F.Cu at (125.3, 120.5)
- added R3: R, Resistor_THT:R_Axial_DIN0309_L9.0mm_D3.2mm_P12.70mm_Horizontal, F.Cu at (124.7, 91.0)
- added R4: R, Resistor_THT:R_Axial_DIN0309_L9.0mm_D3.2mm_P12.70mm_Horizontal, F.Cu at (132.8, 103.7)
- added R5: R, Resistor_THT:R_Axial_DIN0309_L9.0mm_D3.2mm_P12.70mm_Horizontal, F.Cu at (120.6, 103.7)
- added R6: R, Resistor_THT:R_Axial_DIN0309_L9.0mm_D3.2mm_P12.70mm_Horizontal, F.Cu at (116.5, 103.7)
- added R7: R, Resistor_THT:R_Axial_DIN0309_L9.0mm_D3.2mm_P12.70mm_Horizontal, F.Cu at (87.5, 104.9)
- added R8: R, Resistor_THT:R_Axial_DIN0309_L9.0mm_D3.2mm_P12.70mm_Horizontal, F.Cu at (83.7, 92.2)
- added REF**: TestPoint_THTPad_1.5x1.5mm_Drill0.7mm, TestPoint:TestPoint_THTPad_1.5x1.5mm_Drill0.7mm, F.Cu at (146.1, 92.2)
- added REF**: TestPoint_THTPad_1.5x1.5mm_Drill0.7mm, TestPoint:TestPoint_THTPad_1.5x1.5mm_Drill0.7mm, F.Cu at (146.1, 88.3)
- added REF**: TestPoint_THTPad_1.5x1.5mm_Drill0.7mm, TestPoint:TestPoint_THTPad_1.5x1.5mm_Drill0.7mm, F.Cu at (146.1, 95.9)
- A1: moved to B.Cu
- J4: value Conn_01x04 -> Conn_01x03; footprint Connector_PinHeader_2.54mm:PinHeader_1x04_P2.54mm_Vertical -> Connector_PinSocket_2.54mm:PinSocket_1x03_P2.54mm_Vertical
- moved A1 54.4 mm to (89.9, 150.6)
- moved J2 7.16 mm to (133.0, 107.4)
- moved J3 7.15 mm to (129.1, 130.3)
- moved J4 5.01 mm to (146.1, 100.3), turned to 0 degrees
Connections:
- net /R_HIN renamed /Up
- net /_S_LIN renamed /Vn
- net Net-(A1-PadA4) renamed /C10-28
- A1 pad A0: /T_sense -> /ACCEL
- A1 pad A1: /S_sense -> /lu1
- A1 pad A2: /R_sense -> /lw1
- A1 pad A5: /ACCEL -> /TP_OVC1
- A1 pad D0: Net-(A1-D0/RX) -> unconnected-(A1-D0/RX-PadD0)
- A1 pad D1: Net-(A1-D1/TX) -> /HW_5V
- A1 pad D10: Net-(J3-A3) -> /Vp_5V
- A1 pad D11: Net-(J3-A2) -> unconnected-(A1-PadD11)
- A1 pad D12: Net-(J3-A1) -> unconnected-(A1-PadD12)
- A1 pad D13: Net-(J3-A0) -> /Vn_5V
- A1 pad D2: Net-(J2-A5) -> /HU_5V
- A1 pad D3: Net-(J2-A4) -> /HV_5V
- A1 pad D4: Net-(J5-Pin_1) -> /Un_5V
- A1 pad D5: Net-(J5-Pin_2) -> /Up_5V
- A1 pad D6: Net-(J2-A0) -> Net-(J4-Pin_2)
- A1 pad D7: Net-(J2-A2) -> /Dir_5V
- A1 pad D8: Net-(J2-A3) -> /Wn_5V
- A1 pad D9: Net-(J2-A1) -> /Wp_5V
- J1 pad 28: /R_sense -> /lu1
- J1 pad 36: /S_sense -> unconnected-(J1-Pin_36-Pad36)
- J1 pad 38: /T_sense -> /lw1
- J1 pad 59: /S_HIN -> /Vp
- J1 pad 62: /_T_LIN -> /Wn
- J1 pad 64: /_R_LIN -> /Un
- J1 pad 71: /T_HIN -> /Wp
- J1 pad 72: Net-(A1-PadA3) -> /TP_OVC1
- J2 pad 15: /T_HIN -> /Vp
- J2 pad 16: /_T_LIN -> /Wp
- J2 pad 17: /_R_LIN -> /Wn
- J2 pad 19: /S_HIN -> /Un
- J2 pad 2: Net-(J2-A0) -> /Un_5V
- J2 pad 3: Net-(J2-A1) -> /Up_5V
- J2 pad 4: Net-(J2-A2) -> /Wn_5V
- J2 pad 5: Net-(J2-A3) -> /Wp_5V
- J2 pad 6: Net-(J2-A4) -> /Vp_5V
- J2 pad 7: Net-(J2-A5) -> /Vn_5V
- J3 pad 2: Net-(J3-A0) -> /HU_5V
- J3 pad 3: Net-(J3-A1) -> /HW_5V
- J3 pad 4: Net-(J3-A2) -> /HV_5V
- J3 pad 5: Net-(J3-A3) -> /Dir_5V
- J4 pad 2: Net-(A1-D1/TX) -> Net-(J4-Pin_2)
- J4 pad 3: Net-(A1-D0/RX) -> +5V
- J6 pad 4: +3.3V -> +5V
Routing:
- net +5V: track 103.1 -> 246.8 mm
- net +3.3V: track 238.0 -> 97.1 mm, vias 1 -> 0
- net /TP_OVC1: track 0.00 -> 135.4 mm
- net Net-(A1-PadA3): track 137.3 -> 8.69 mm
- net /HW_5V: track 0.00 -> 85.5 mm
- net /HV_5V: track 0.00 -> 85.1 mm, vias 0 -> 1
- net /Dir_5V: track 0.00 -> 84.1 mm, vias 0 -> 1
- net /HU_5V: track 0.00 -> 82.8 mm
- net /lw1: track 0.00 -> 75.6 mm
- net /S_sense: track 61.7 -> 0.00 mm
- net /T_sense: track 58.7 -> 0.00 mm, vias 1 -> 0
- net /R_sense: track 55.6 -> 0.00 mm
- net /lu1: track 0.00 -> 53.2 mm
- net /_T_LIN: track 51.3 -> 0.00 mm
- net /Vp: track 0.00 -> 49.9 mm, vias 0 -> 1
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Other:
- outline, holes or cut-outs redrawn
- board text added: "3V3"
- board text added: "5V"
- board text added: "5V1"
- board text added: "ACCEL"
- board text added: "D6"
- board text added: "Direction"
- board text added: "GND"
- board text added: "HU"
- board text added: "HU_5V"
- board text added: "HV"
- board text added: "HV_5V"
- board text added: "HW"
- board text added: "HW_5V"
- board text added: "SCL"
- board text added: "SDA"
- board text added: "Un"
- board text added: "Un_5V"
- board text added: "Up"
- board text added: "Up_5V"
- board text added: "VIN"
- board text added: "Vdc"
- board text added: "Vn"
- board text added: "Vn_5V"
- board text added: "Vp"
- board text added: "Vp_5V"
- board text added: "Wn"
- board text added: "Wn_5V"
- board text added: "Wp"
- board text added: "Wp_5V"
- board text added: "lu1"
- board text added: "lw1"
- board text added: "インバータ・キット2 Arduino Ver 0.1"

Commit message: 0122
Connections:
- J1 pad 19: unconnected-(J1-Pin_19-Pad19) -> GND
- J1 pad 20: unconnected-(J1-Pin_20-Pad20) -> GND
- J1 pad 22: unconnected-(J1-Pin_22-Pad22) -> GND
- J1 pad 47: unconnected-(J1-Pad47) -> GND
- J1 pad 58: unconnected-(J1-Pad58) -> GND
- J1 pad 70: unconnected-(J1-Pad70) -> GND
- J1 pad 8: unconnected-(J1-Pin_8-Pad8) -> GND
Routing:
- net GND: track 0.00 -> 9.97 mm
- net /HU: track 92.4 -> 93.3 mm
Other:
- board text added: "インバータ・キット2 Arduino Ver 0.2"
- board text removed: "インバータ・キット2 Arduino Ver 0.1"

Commit message: ver0.3
Parts:
- removed R7, R8: R, Resistor_THT:R_Axial_DIN0309_L9.0mm_D3.2mm_P12.70mm_Horizontal
Connections:
- A1 pad A3: Net-(A1-PadA3) -> Net-(J1-Pin_30)
- J1 pad 30: unconnected-(J1-Pin_30-Pad30) -> Net-(J1-Pin_30)
Routing:
- net Net-(J1-Pin_30): track 0.00 -> 63.2 mm, vias 0 -> 1
- net Net-(A1-PadA3): track 8.69 -> 0.00 mm
- net /VIN: track 44.7 -> 39.8 mm
- net /Vn: track 55.6 -> 56.4 mm
- net /Dir_5V: track 84.1 -> 83.5 mm
Other:
- board text added: "インバータ・キット2 Arduino Ver 0.3"
- board text removed: "インバータ・キット2 Arduino Ver 0.2"

Commit message: 0209
Routing:
- net GND: track 9.97 -> 16.6 mm, vias 13 -> 14
- net +3.3V: track 97.1 -> 97.8 mm

Commit message: ver 0.4 (add LDO)
Parts:
- removed J2, J3: AE-LLCNV8-DIP20, Library:AE-LLCNV8-DIP
- added IC1: AZ1084CD-5.0TRG1, samacsys:AZ1084CD50TRG1, F.Cu at (111.0, 135.8)
- moved R6 24.3 mm to (137.8, 115.6), turned to 180 degrees
- moved R3 20.7 mm to (137.3, 107.4), turned to 180 degrees
- moved R5 12.9 mm to (130.9, 111.5), turned to 180 degrees
- moved R1 10.2 mm to (137.3, 96.5), turned to 180 degrees
- moved R4 5.47 mm to (137.3, 100.6), turned to 180 degrees
- moved R2 3.25 mm to (128.4, 121.5), turned to 180 degrees
Connections:
- net Net-(J1-Pin_30) renamed /BATT
- A1 pad 3V3: +3.3V -> unconnected-(A1-3.3V-Pad3V3)
- A1 pad 5V1: +5V -> unconnected-(A1-5V-Pad5V1)
- A1 pad AREF: +3.3V -> +5V
- A1 pad D1: /HW_5V -> /HW
- A1 pad D10: /Vp_5V -> /Vp
- A1 pad D13: /Vn_5V -> /Vn
- A1 pad D2: /HU_5V -> /HU
- A1 pad D3: /HV_5V -> /HV
- A1 pad D4: /Un_5V -> /Un
- A1 pad D5: /Up_5V -> /Up
- A1 pad D7: /Dir_5V -> /Dir
- A1 pad D8: /Wn_5V -> /Wn
- A1 pad D9: /Wp_5V -> /Wp
- J1 pad 16: +3.3V -> +5V
- J1 pad 41: /Direction -> /Dir
- R1 pad 1: +5V -> /Un
- R1 pad 2: /Un_5V -> +5V
- R2 pad 1: +5V -> /Vn
- R2 pad 2: /Vn_5V -> +5V
- R3 pad 1: +5V -> /Wn
- R3 pad 2: /Wn_5V -> +5V
- R4 pad 1: /Up_5V -> /Up
- R5 pad 1: /Wp_5V -> /Wp
- R6 pad 1: /Vp_5V -> /Vp
- REF** pad 1: /HU_5V -> /HU
- REF** pad 1: /HW_5V -> /HW
- REF** pad 1: /HV_5V -> /HV
Routing:
- net +3.3V: track 97.8 -> 0.00 mm
- net /Direction: track 95.5 -> 0.00 mm
- net +5V: track 246.8 -> 154.2 mm
- net /HW_5V: track 85.3 -> 0.00 mm
- net /HV_5V: track 84.7 -> 0.00 mm, vias 1 -> 0
- net /Dir_5V: track 83.5 -> 0.00 mm, vias 1 -> 0
- net /HU_5V: track 82.7 -> 0.00 mm
- net /HW: track 23.9 -> 69.9 mm
- net /HV: track 30.4 -> 66.9 mm
- net /Vn_5V: track 32.8 -> 0.00 mm
- net /Vp_5V: track 29.7 -> 0.00 mm
- net /Un: track 34.9 -> 63.1 mm, vias 1 -> 0
- net /Wp_5V: track 25.1 -> 0.00 mm
- net /HU: track 93.3 -> 118.2 mm, vias 0 -> 1
- net /VIN: track 39.8 -> 63.6 mm
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Other:
- board text added: "BATT"
- board text added: "インバータ・キット2 Arduino Ver 0.4"
- board text removed: "Direction"
- board text removed: "HU_5V"
- board text removed: "HV_5V"
- board text removed: "HW_5V"
- board text removed: "Un_5V"
- board text removed: "Up_5V"
- board text removed: "Vdc"
- board text removed: "Vn"
- board text removed: "Vn_5V"
- board text removed: "Vp_5V"
- board text removed: "Wn_5V"
- board text removed: "Wp_5V"
- board text removed: "インバータ・キット2 Arduino Ver 0.3"

Commit message: 0214
Parts:
- added J2: Conn_01x06_Socket, Connector_PinHeader_2.54mm:PinHeader_1x06_P2.54mm_Vertical, F.Cu at (110.2, 80.1)
- added SW1: SW_SPDT, Connector_PinHeader_2.54mm:PinHeader_1x03_P2.54mm_Vertical, F.Cu at (85.9, 83.5)
- added SW2: SW_SPDT, Connector_PinHeader_2.54mm:PinHeader_1x03_P2.54mm_Vertical, F.Cu at (85.9, 95.6)
- added TP1: TestPoint, TestPoint:TestPoint_Pad_D1.5mm, F.Cu at (88.1, 92.2)
Connections:
- A1 pad 5V2: unconnected-(A1-SPI_5V-Pad5V2) -> Net-(A1-SPI_5V)
- A1 pad D11: unconnected-(A1-PadD11) -> Net-(SW1-B)
- A1 pad D12: unconnected-(A1-PadD12) -> Net-(SW2-B)
- A1 pad GND4: unconnected-(A1-SPI_GND-PadGND4) -> GND
- A1 pad MISO: unconnected-(A1-SPI_MISO-PadMISO) -> Net-(A1-SPI_MISO)
- A1 pad MOSI: unconnected-(A1-SPI_MOSI-PadMOSI) -> Net-(A1-SPI_MOSI)
- A1 pad RST2: unconnected-(A1-SPI_RESET-PadRST2) -> Net-(A1-SPI_RESET)
- A1 pad SCK: unconnected-(A1-SPI_SCK-PadSCK) -> Net-(A1-SPI_SCK)
Routing:
- net Net-(SW2-B): track 0.00 -> 94.2 mm
- net Net-(SW1-B): track 0.00 -> 84.2 mm
- net Net-(A1-SPI_5V): track 0.00 -> 25.4 mm
- net +5V: track 154.2 -> 175.0 mm
- net Net-(A1-SPI_MISO): track 0.00 -> 10.2 mm
- net Net-(A1-SPI_RESET): track 0.00 -> 9.68 mm
- net Net-(A1-SPI_SCK): track 0.00 -> 7.84 mm
- net Net-(A1-SPI_MOSI): track 0.00 -> 5.34 mm
- net GND: track 0.00 -> 4.58 mm, vias 15 -> 19
- net /BATT: track 73.9 -> 78.2 mm
- net /ACCEL: track 63.2 -> 60.8 mm
- net /C10-28: track 120.7 -> 122.7 mm
- net /Vn: track 80.5 -> 78.7 mm
- net /HU: track 118.2 -> 120.0 mm, vias 1 -> 0
- net /TP_OVC1: track 132.6 -> 133.9 mm
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Other:
- board text added: "5V2"
- board text added: "AREF"
- board text added: "D11"
- board text added: "D12"
- board text added: "Dir"
- board text added: "MISO"
- board text added: "MOSI"
- board text added: "RST2"
- board text added: "SCK"
- board text added: "Vn"
- board text removed: "5V1"

Commit message: 0220
Parts:
- added C1: C, Capacitor_SMD:C_0603_1608Metric_Pad1.08x0.95mm_HandSolder, F.Cu at (121.7, 138.4)
- added C2: C_Polarized, Capacitor_THT:CP_Radial_D8.0mm_P3.50mm, F.Cu at (119.0, 143.1)
- added C3: C, Capacitor_SMD:C_0603_1608Metric_Pad1.08x0.95mm_HandSolder, F.Cu at (104.8, 140.5)
- added C4: C_Polarized, Capacitor_THT:CP_Radial_D8.0mm_P3.50mm, F.Cu at (109.1, 143.1)
- added J3: Conn_01x01_Pin, Connector_PinHeader_2.54mm:PinHeader_1x01_P2.54mm_Vertical, F.Cu at (84.8, 159.8)
- added JP1: SolderJumper_2_Bridged, Jumper:SolderJumper-2_P1.3mm_Bridged_Pad1.0x1.5mm, F.Cu at (85.9, 106.8)
- added R7: R, Resistor_SMD:R_0603_1608Metric_Pad0.98x0.95mm_HandSolder, F.Cu at (85.9, 104.4)
Connections:
- A1 pad A0: /ACCEL -> Net-(JP1-A)
Routing:
- net +5V: track 175.0 -> 190.3 mm
- net Net-(JP1-A): track 0.00 -> 14.0 mm
- net /VIN: track 63.6 -> 70.4 mm
- net GND: vias 19 -> 16
