File: Arduino_CQbrushless.kicad_pcb (KiCad board)
At the start: 2 copper layers, 72.6 x 85.1 mm, 25 parts, among them IC1 AZ1084CD-5.0TRG1, J1 Nucleo_F302R8, J2 Conn_01x06_Socket, J3 Conn_01x01_Pin, J4 Conn_01x03, J6 Conn_01x04, SW1 SW_SPDT, SW2 SW_SPDT

Commit message: 0416
Parts:
- C1: footprint Capacitor_SMD:C_0603_1608Metric_Pad1.08x0.95mm_HandSolder -> Capacitor_SMD:C_0805_2012Metric_Pad1.18x1.45mm_HandSolder
- moved C1 0.25 mm to (121.9, 138.4)
Other:
- board text added: "インバータ・キット2 Arduino Ver 0.5"
- board text removed: "インバータ・キット2 Arduino Ver 0.4"
